File: V4.0.kicad_sch (KiCad schematic)
At the start: 67 parts, among them J1 USB_A_Stacked, J2 USB-C-PD-HRO, J3 USB-C-PD-HRO, J4 XT60, J5 Conn_01x06_Female, Q1 IPG20N04S4-08, Q2 IPG20N04S4-08, Q3 IPG20N04S4-08, Q4 IPG20N04S4-08, Q5 2SJ168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

Commit message: fixed parameter
Parts:
- C14: value 2.2nf -> (none)
- R10: value 27K -> (none); footprint Resistor_SMD:R_0805_2012Metric -> (none)
- R12: value 100R -> (none)
- R4: value 10K -> (none); footprint Resistor_SMD:R_0805_2012Metric -> (none)
Changed lines of the file:
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@@
   (symbol (lib_id "Device:C") (at 175.895 114.935 90) (unit 1)
     (in_bom yes) (on_board yes) (fields_autoplaced)
-    (property "Reference" "C14" (id 0) (at 175.895 107.95 90))
-    (property "Value" "2.2nf" (id 1) (at 175.895 110.49 90))
+    (property "Reference" "C14" (id 0) (at 175.895 109.0762 90))
+    (property "Value" "" (id 1) (at 175.895 111.6131 90))
     (property "Footprint" "Capacitor_SMD:C_0805_2012Metric" (id 2) (at 179.705 113.9698 0)
       (effects (font (size 1.27 1.27)) hide)
@@
       (effects (font (size 1.27 1.27)) (justify right))
     )
-    (property "Value" "10K" (id 1) (at 144.78 97.7899 0)
-      (effects (font (size 1.27 1.27)) (justify right))
-    )
-    (property "Footprint" "Resistor_SMD:R_0805_2012Metric" (id 2) (at 142.875 96.52 0)
+    (property "Value" "" (id 1) (at 144.78 97.7899 0)
+      (effects (font (size 1.27 1.27)) (justify right))
+    )
+    (property "Footprint" "" (id 2) (at 142.875 96.52 0)
       (effects (font (size 1.27 1.27)) hide)
     )
@@
     (in_bom yes) (on_board yes)
     (property "Reference" "R12" (id 0) (at 200.025 95.885 90))
-    (property "Value" "100R" (id 1) (at 195.58 95.885 90))
+    (property "Value" "" (id 1) (at 195.58 95.885 90))
     (property "Footprint" "Resistor_SMD:R_0805_2012Metric" (id 2) (at 198.12 100.203 90)
       (effects (font (size 1.27 1.27)) hide)
@@
   )
   (symbol (lib_id "Device:R") (at 198.12 84.455 90) (unit 1)
-    (in_bom yes) (on_board yes) (fields_autoplaced)
-    (property "Reference" "R10" (id 0) (at 198.12 76.2 90))
-    (property "Value" "27K" (id 1) (at 198.12 78.74 90))
-    (property "Footprint" "Resistor_SMD:R_0805_2012Metric" (id 2) (at 198.12 81.28 90))
+    (in_bom yes) (on_board yes)
+    (property "Reference" "R10" (id 0) (at 198.12 77.2024 90))
+    (property "Value" "" (id 1) (at 198.12 85.09 90))
+    (property "Footprint" "" (id 2) (at 198.12 82.2762 90)
+      (effects (font (size 1.27 1.27)) hide)
+    )
     (property "Datasheet" "~" (id 3) (at 198.12 84.455 0)
       (effects (font (size 1.27 1.27)) hide)
@@
     )
     (path "/223eb1f0-eeb3-492d-8711-17508cf24aee"
-      (reference "C14") (unit 1) (value "2.2nf") (footprint "Capacitor_SMD:C_0805_2012Metric")
+      (reference "C14") (unit 1) (value "2.2uf") (footprint "Capacitor_SMD:C_0805_2012Metric")
     )
     (path "/2bf4ec40-73c7-48e0-8bc1-c2f040c68678"
@@
     )
     (path "/6115a883-b57c-4732-87bd-6c703cca8710"
-      (reference "R4") (unit 1) (value "10K") (footprint "Resistor_SMD:R_0805_2012Metric")
+      (reference "R4") (unit 1) (value "20R") (footprint "Resistor_SMD:R_0805_2012Metric")
     )
     (path "/decbffc5-e135-4f19-b7fa-4e8ffa988e66"
@@
     )
     (path "/8825542a-d729-4e2a-a91e-989edbffbd8d"
-      (reference "R12") (unit 1) (value "100R") (footprint "Resistor_SMD:R_0805_2012Metric")
+      (reference "R12") (unit 1) (value "27K") (footprint "Resistor_SMD:R_0805_2012Metric")
     )
     (path "/06e1469d-2d38-4720-a9e3-0856566eefca"
